File: PCB/EPICS_Connect4.kicad_sch (KiCad schematic)
At the start: 25 parts, among them J1 Power, J4 EndA, J5 EndB, J6 LEDA, J7 LEDB, J8 Motor

Commit message: Update EPICS_Connect4 KiCad project
Co-Authored-By: Claude Sonnet 5 <noreply@anthropic.com>
Parts:
- removed C1: 100uF, Capacitor_SMD:CP_Elec_6.3x5.9, symbol Device:C_Polarized_Small
- added C1: 10uF, Capacitor_SMD:C_0805_2012Metric, symbol Device:C_Small
- added D6: LED_Small, LED_SMD:LED_0805_2012Metric, symbol Device:LED_Small
- added R22, R23: 330, Resistor_SMD:R_0603_1608Metric, symbol Device:R_Small
- added SYM1: Logo_Open_Hardware_Large, Library:S_Silk_Logo, symbol Graphic:Logo_Open_Hardware_Large
- J1: footprint Connector_Molex:Molex_Micro-Fit_3.0_43650-0215_1x02_P3.00mm_Vertical -> Connector_Molex:Molex_Micro-Fit_3.0_43650-0200_1x02_P3.00mm_Horizontal
- J4, J5: footprint Connector_JST:JST_PH_S2B-PH-K_1x02_P2.00mm_Horizontal -> Connector_JST:JST_PH_B2B-PH-K_1x02_P2.00mm_Vertical
Connections:
- net +12V: now also R22.1
- net GND: now also C1.2, R23.2
- net Power Regulators/+VIN: now also C1.1
- new net: D6.2 (A), R22.2
- new net: D6.1 (K), R23.1
Other:
- sheet Motor Acuator ports: added M1[3..0]; removed M1
- moved on the sheet: J8
