File: PCB/EPICS_Connect4.kicad_sch (KiCad schematic)
At the start: 29 parts, among them J1 Power, J4 EndA, J5 EndB, J6 LEDA, J7 LEDB, J8 Motor

Commit message: Update PCB layout
Co-Authored-By: Claude Sonnet 5 <noreply@anthropic.com>
Parts:
- removed D6: LED_Small, LED_SMD:LED_0805_2012Metric, symbol Device:LED_Small
- removed R22, R23: 330, Resistor_SMD:R_0603_1608Metric, symbol Device:R_Small
