File: PCB/EPICS_Connect4.kicad_pcb (KiCad board)
At the start: 4 copper layers, 50 x 60 mm, 90 parts, among them J1 Power, J2 TC2030, J3 USB_C_Receptacle_USB2.0_14P, J4 EndA, J5 EndB, J6 LEDA, J7 LEDB, J8 Motor, SW1 ESP.RST, SW2 ESP.BOOT, U1 TPS54202DDC, U2 AP2205-5, U3 STM32G474CBTx, U4 SN74AHCT1G125DBVR, U5 SN74AHCT1G125DBVR, U6 ESP32-C3-WROOM-02, U7 USBLC6-2SC6, U8 TMC2209

Commit message: last_12V
Parts:
- J4, J5: footprint Connector_JST:JST_PH_B2B-PH-K_1x02_P2.00mm_Vertical -> Connector_JST:JST_EH_B2B-EH-A_1x02_P2.50mm_Vertical
- moved J4 0.75 mm to (131.2, 93.0)
- moved J5 0.75 mm to (131.2, 100.0)
- moved J1 0.50 mm to (159.0, 125.5)
- moved C1 0.49 mm to (156.5, 131.2)
- moved D1 0.49 mm to (153.5, 127.8)
- moved F1 0.49 mm to (156.5, 127.0)
- moved D2 0.25 mm to (148.6, 92.0)
- moved R13 0.25 mm to (155.0, 92.8)
- moved R9 0.25 mm to (166.1, 99.2)
Routing:
- net Net-(J1-Pin_1): track 2.51 -> 0.00 mm
- net GND: track 37.5 -> 35.1 mm, vias 106 -> 110
- net /ESP32 Weblink/IO9: track 14.6 -> 13.8 mm
- net /ESP32 Weblink/EN: track 27.4 -> 26.6 mm
- net /STM32 Controller/END.B: track 1.60 -> 2.35 mm
- net /STM32 Controller/END.A: track 1.60 -> 2.35 mm
- net +3V3: track 51.2 -> 50.4 mm
- net +5V: track 24.8 -> 24.2 mm
- added copper zone on F.Cu, net Net-(J1-Pin_1)
Other:
- outline, holes or cut-outs redrawn
