File: PCB/EPICS_Connect4.kicad_pcb (KiCad board)
At the start: 4 copper layers, 50 x 60 mm, 84 parts, among them J1 +5V, J2 +12V, J3 EndA, J4 EndB, J5 LEDA, J6 LEDB, J7 MOTOR, J8 USB_C_Receptacle_USB2.0_14P, J9 TC2030, SW1 ESP.RST, SW2 ESP.BOOT, U1 TPS54202DDC, U2 SN74AHCT1G125DBVR, U3 SN74AHCT1G125DBVR, U4 USBLC6-2SC6, U5 TMC2209, U6 STM32G474CBTx, U7 ESP32-C3-WROOM-02

Commit message: Ready for Fab
Parts:
- C1, C2: value 10uF -> 22uF
- moved SYM1 1.58 mm to (160.0, 122.0)
- renumbered U6 to U2, U2 to U3, U3 to U4, U7 to U5, U4 to U6, U5 to U7
Other:
- board text added: "EPICS"
- board text removed: "EPICS Klondike"

Commit message: text fixes
Parts:
- moved SYM1 0.50 mm to (160.0, 122.5)
Other:
- board text added: ":)"
