File: PCB/esp32.kicad_sch (KiCad schematic)
At the start: 18 parts, among them J3 USB_C_Receptacle_USB2.0_14P, SW1 ESP.RST, SW2 ESP.BOOT, U5 ESP32-C3-WROOM-02, U6 USBLC6-2SC6

Commit message: Update EPICS_Connect4 KiCad project
Co-Authored-By: Claude Sonnet 5 <noreply@anthropic.com>
Parts:
- SW1, SW2: footprint Button_Switch_THT:SW_PUSH_6mm_H4.3mm -> Button_Switch_SMD:SW_Push_1P1T_NO_CK_KMR2
- renumbered C20 to C19, C19 to C20, U5 to U6, U6 to U7
Changed lines of the file:
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@@
 		(dnp no)
 		(fields_autoplaced yes)
-		(property "Reference" "C19"
+		(property "Reference" "C20"
 			(at 180.34 77.4699 0)
 			(show_name no)
@@
 			(project "EPICS_Connect4"
 				(path "/7f359823-7e50-4056-8b4f-ffb6c29ecc64/df1c4d5a-0179-43c9-baee-07d6baf032a1"
-					(reference "C19")
+					(reference "C20")
 					(unit 1)
 				)
@@
 		(dnp no)
 		(fields_autoplaced yes)
-		(property "Reference" "#PWR?"
+		(property "Reference" "#PWR038"
 			(at 60.96 133.35 0)
 			(hide yes)
@@
 			(project "EPICS_Connect4"
 				(path "/7f359823-7e50-4056-8b4f-ffb6c29ecc64/df1c4d5a-0179-43c9-baee-07d6baf032a1"
-					(reference "#PWR?")
+					(reference "#PWR038")
 					(unit 1)
 				)
@@
 		(dnp no)
 		(fields_autoplaced yes)
-		(property "Reference" "#PWR?"
+		(property "Reference" "#PWR039"
 			(at 88.9 133.35 0)
 			(hide yes)
@@
 			(project "EPICS_Connect4"
 				(path "/7f359823-7e50-4056-8b4f-ffb6c29ecc64/df1c4d5a-0179-43c9-baee-07d6baf032a1"
-					(reference "#PWR?")
+					(reference "#PWR039")
 					(unit 1)
 				)
@@
 		(dnp no)
 		(fields_autoplaced yes)
-		(property "Reference" "#PWR?"
+		(property "Reference" "#PWR047"
 			(at 177.8 87.63 0)
 			(hide yes)
@@
 			(project "EPICS_Connect4"
 				(path "/7f359823-7e50-4056-8b4f-ffb6c29ecc64/df1c4d5a-0179-43c9-baee-07d6baf032a1"
-					(reference "#PWR?")
+					(reference "#PWR047")
 					(unit 1)
 				)
@@
 		(dnp no)
 		(fields_autoplaced yes)
-		(property "Reference" "U5"
+		(property "Reference" "U6"
 			(at 205.3433 86.36 0)
 			(show_name no)
@@
 			(project "EPICS_Connect4"
 				(path "/7f359823-7e50-4056-8b4f-ffb6c29ecc64/df1c4d5a-0179-43c9-baee-07d6baf032a1"
-					(reference "U5")
+					(reference "U6")
 					(unit 1)
 				)
@@
 		(in_pos_files yes)
 		(dnp no)
-		(property "Reference" "C20"
+		(property "Reference" "C19"
 			(at 175.26 95.2499 0)
 			(show_name no)
@@
 			(project "EPICS_Connect4"
 				(path "/7f359823-7e50-4056-8b4f-ffb6c29ecc64/df1c4d5a-0179-43c9-baee-07d6baf032a1"
-					(reference "C20")
+					(reference "C19")
 					(unit 1)
 				)
@@
 		(dnp no)
 		(fields_autoplaced yes)
-		(property "Reference" "#PWR?"
+		(property "Reference" "#PWR050"
 			(at 228.6 118.11 0)
 			(hide yes)
@@
 			(project "EPICS_Connect4"
 				(path "/7f359823-7e50-4056-8b4f-ffb6c29ecc64/df1c4d5a-0179-43c9-baee-07d6baf032a1"
-					(reference "#PWR?")
+					(reference "#PWR050")
 					(unit 1)
 				)
@@
 		(dnp no)
 		(fields_autoplaced yes)
-		(property "Reference" "#PWR?"
+		(property "Reference" "#PWR044"
 			(at 152.4 113.03 0)
 			(hide yes)
@@
 			(project "EPICS_Connect4"
 				(path "/7f359823-7e50-4056-8b4f-ffb6c29ecc64/df1c4d5a-0179-43c9-baee-07d6baf032a1"
-					(reference "#PWR?")
+					(reference "#PWR044")
 					(unit 1)
 				)
@@
 		(dnp no)
 		(fields_autoplaced yes)
-		(property "Reference" "#PWR?"
+		(property "Reference" "#PWR046"
 			(at 177.8 80.01 0)
 			(hide yes)
@@
 			(project "EPICS_Connect4"
 				(path "/7f359823-7e50-4056-8b4f-ffb6c29ecc64/df1c4d5a-0179-43c9-baee-07d6baf032a1"
-					(reference "#PWR?")
+					(reference "#PWR046")
 					(unit 1)
 				)
@@
 			)
 		)
-		(property "Footprint" "Button_Switch_THT:SW_PUSH_6mm_H4.3mm"
+		(property "Footprint" "Button_Switch_SMD:SW_Push_1P1T_NO_CK_KMR2"
 			(at 134.62 119.38 0)
 			(hide yes)
@@
 		(dnp no)
 		(fields_autoplaced yes)
-		(property "Reference" "#PWR?"
+		(property "Reference" "#PWR042"
 			(at 139.7 130.81 0)
 			(hide yes)
@@
 			(project "EPICS_Connect4"
 				(path "/7f359823-7e50-4056-8b4f-ffb6c29ecc64/df1c4d5a-0179-43c9-baee-07d6baf032a1"
-					(reference "#PWR?")
+					(reference "#PWR042")
 					(unit 1)
 				)
@@
 		(dnp no)
 		(fields_autoplaced yes)
-		(property "Reference" "#PWR?"
+		(property "Reference" "#PWR037"
 			(at 53.34 133.35 0)
 			(hide yes)
@@
 			(project "EPICS_Connect4"
 				(path "/7f359823-7e50-4056-8b4f-ffb6c29ecc64/df1c4d5a-0179-43c9-baee-07d6baf032a1"
-					(reference "#PWR?")
+					(reference "#PWR037")
 					(unit 1)
 				)
@@
 		(dnp no)
 		(fields_autoplaced yes)
-		(property "Reference" "#PWR?"
+		(property "Reference" "#PWR045"
 			(at 152.4 130.81 0)
 			(hide yes)
@@
 			(project "EPICS_Connect4"
 				(path "/7f359823-7e50-4056-8b4f-ffb6c29ecc64/df1c4d5a-0179-43c9-baee-07d6baf032a1"
-					(reference "#PWR?")
+					(reference "#PWR045")
 					(unit 1)
 				)
@@
 		(dnp no)
 		(fields_autoplaced yes)
-		(property "Reference" "#PWR?"
+		(property "Reference" "#PWR043"
 			(at 152.4 95.25 0)
 			(hide yes)
@@
 			(project "EPICS_Connect4"
 				(path "/7f359823-7e50-4056-8b4f-ffb6c29ecc64/df1c4d5a-0179-43c9-baee-07d6baf032a1"
-					(reference "#PWR?")
+					(reference "#PWR043")
 					(unit 1)
 				)
@@
 			)
 		)
-		(property "Footprint" "Button_Switch_THT:SW_PUSH_6mm_H4.3mm"
+		(property "Footprint" "Button_Switch_SMD:SW_Push_1P1T_NO_CK_KMR2"
 			(at 147.32 119.38 0)
 			(hide yes)
@@
 		(dnp no)
 		(fields_autoplaced yes)
-		(property "Reference" "#PWR?"
+		(property "Reference" "#PWR049"
 			(at 203.2 140.97 0)
 			(hide yes)
@@
 			(project "EPICS_Connect4"
 				(path "/7f359823-7e50-4056-8b4f-ffb6c29ecc64/df1c4d5a-0179-43c9-baee-07d6baf032a1"
-					(reference "#PWR?")
+					(reference "#PWR049")
 					(unit 1)
 				)
@@
 		(dnp no)
 		(fields_autoplaced yes)
-		(property "Reference" "#PWR?"
+		(property "Reference" "#PWR041"
 			(at 139.7 113.03 0)
 			(hide yes)
@@
 			(project "EPICS_Connect4"
 				(path "/7f359823-7e50-4056-8b4f-ffb6c29ecc64/df1c4d5a-0179-43c9-baee-07d6baf032a1"
-					(reference "#PWR?")
+					(reference "#PWR041")
 					(unit 1)
 				)
@@
 		(dnp no)
 		(fields_autoplaced yes)
-		(property "Reference" "#PWR?"
+		(property "Reference" "#PWR040"
 			(at 139.7 95.25 0)
 			(hide yes)
@@
 			(project "EPICS_Connect4"
 				(path "/7f359823-7e50-4056-8b4f-ffb6c29ecc64/df1c4d5a-0179-43c9-baee-07d6baf032a1"
-					(reference "#PWR?")
+					(reference "#PWR040")
 					(unit 1)
 				)
@@
 		(in_pos_files yes)
 		(dnp no)
-		(property "Reference" "U6"
+		(property "Reference" "U7"
 			(at 90.5511 95.25 0)
 			(show_name no)
@@
 			(project "EPICS_Connect4"
 				(path "/7f359823-7e50-4056-8b4f-ffb6c29ecc64/df1c4d5a-0179-43c9-baee-07d6baf032a1"
-					(reference "U6")
+					(reference "U7")
 					(unit 1)
 				)
@@
 		(dnp no)
 		(fields_autoplaced yes)
-		(property "Reference" "#PWR?"
+		(property "Reference" "#PWR048"
 			(at 177.8 105.41 0)
 			(hide yes)
@@
 			(project "EPICS_Connect4"
 				(path "/7f359823-7e50-4056-8b4f-ffb6c29ecc64/df1c4d5a-0179-43c9-baee-07d6baf032a1"
-					(reference "#PWR?")
+					(reference "#PWR048")
 					(unit 1)
 				)

Commit message: Update PCB layout, ESP32 schematic, and fab outputs
Co-Authored-By: Claude Sonnet 5 <noreply@anthropic.com>
Parts:
- U6: footprint RF_Module:ESP32-C3-WROOM-02 -> Library:ESP32-C3-WROOM-02_Modified
Changed lines of the file:
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@@
 			)
 		)
-		(property "Footprint" "RF_Module:ESP32-C3-WROOM-02"
+		(property "Footprint" "Library:ESP32-C3-WROOM-02_Modified"
 			(at 203.2 111.125 0)
 			(hide yes)

Commit message: Minor PCB updates
Co-Authored-By: Claude Sonnet 5 <noreply@anthropic.com>
Parts:
- added TP12: IO0, TestPoint:TestPoint_Pad_2.0x2.0mm, symbol Connector:TestPoint
- added TP13: IO1, TestPoint:TestPoint_Pad_2.0x2.0mm, symbol Connector:TestPoint
- added TP14: IO3, TestPoint:TestPoint_Pad_2.0x2.0mm, symbol Connector:TestPoint
Connections:
- net IO3: now reaches U6.15 (IO3)
- net IO3: now also TP14.1
- net IO1: now reaches U6.17 (IO1)
- net IO1: now also TP13.1
- net IO0: now reaches U6.18 (IO0)
- net IO0: now also TP12.1
- no-connect marks 5 -> 2
Other:
- note added: "EXTRA GPIO OUTPUTS"

Commit message: Swap Molex connector 3D model to 43650-0215
Co-Authored-By: Claude Opus 5.5 <noreply@anthropic.com>
Parts:
- TP6: renamed from TP12; now left out of the parts list
- TP7: renamed from TP13; now left out of the parts list
- TP8: renamed from TP14; now left out of the parts list
- renumbered C20 to C17, C21 to C18, D3 to D5, J3 to J8, R14 to R13, R16 to R14, R17 to R15, R15 to R16, R13 to R17, U7 to U4, U6 to U7
Changed lines of the file:
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@@
 		(dnp no)
 		(fields_autoplaced yes)
-		(property "Reference" "C20"
+		(property "Reference" "C17"
 			(at 180.34 77.4699 0)
 			(show_name no)
@@
 			(project "EPICS_Connect4"
 				(path "/7f359823-7e50-4056-8b4f-ffb6c29ecc64/df1c4d5a-0179-43c9-baee-07d6baf032a1"
-					(reference "C20")
+					(reference "C17")
 					(unit 1)
 				)
@@
 		(dnp no)
 		(fields_autoplaced yes)
-		(property "Reference" "#PWR038"
+		(property "Reference" "#PWR036"
 			(at 60.96 133.35 0)
 			(hide yes)
@@
 			(project "EPICS_Connect4"
 				(path "/7f359823-7e50-4056-8b4f-ffb6c29ecc64/df1c4d5a-0179-43c9-baee-07d6baf032a1"
-					(reference "#PWR038")
+					(reference "#PWR036")
 					(unit 1)
 				)
@@
 		(body_style 1)
 		(exclude_from_sim no)
-		(in_bom yes)
+		(in_bom no)
 		(on_board yes)
 		(in_pos_files yes)
 		(dnp no)
-		(property "Reference" "TP12"
+		(property "Reference" "TP6"
 			(at 139.7 69.85 0)
 			(show_name no)
@@
 			(project "EPICS_Connect4"
 				(path "/7f359823-7e50-4056-8b4f-ffb6c29ecc64/df1c4d5a-0179-43c9-baee-07d6baf032a1"
-					(reference "TP12")
+					(reference "TP6")
 					(unit 1)
 				)
@@
 		(dnp no)
 		(fields_autoplaced yes)
-		(property "Reference" "R16"
+		(property "Reference" "R14"
 			(at 142.24 92.7099 0)
 			(show_name no)
@@
 			(project "EPICS_Connect4"
 				(path "/7f359823-7e50-4056-8b4f-ffb6c29ecc64/df1c4d5a-0179-43c9-baee-07d6baf032a1"
-					(reference "R16")
+					(reference "R14")
 					(unit 1)
 				)
@@
 		(dnp no)
 		(fields_autoplaced yes)
-		(property "Reference" "#PWR039"
+		(property "Reference" "#PWR037"
 			(at 88.9 133.35 0)
 			(hide yes)
@@
 			(project "EPICS_Connect4"
 				(path "/7f359823-7e50-4056-8b4f-ffb6c29ecc64/df1c4d5a-0179-43c9-baee-07d6baf032a1"
-					(reference "#PWR039")
+					(reference "#PWR037")
 					(unit 1)
 				)
@@
 		(dnp no)
 		(fields_autoplaced yes)
-		(property "Reference" "#PWR047"
+		(property "Reference" "#PWR045"
 			(at 177.8 87.63 0)
 			(hide yes)
@@
 			(project "EPICS_Connect4"
 				(path "/7f359823-7e50-4056-8b4f-ffb6c29ecc64/df1c4d5a-0179-43c9-baee-07d6baf032a1"
-					(reference "#PWR047")
+					(reference "#PWR045")
 					(unit 1)
 				)
@@
 		(dnp no)
 		(fields_autoplaced yes)
-		(property "Reference" "U6"
+		(property "Reference" "U7"
 			(at 205.3433 86.36 0)
 			(show_name no)
@@
 			(project "EPICS_Connect4"
 				(path "/7f359823-7e50-4056-8b4f-ffb6c29ecc64/df1c4d5a-0179-43c9-baee-07d6baf032a1"
-					(reference "U6")
+					(reference "U7")
 					(unit 1)
 				)
@@
 		(in_pos_files yes)
 		(dnp no)
-		(property "Reference" "R14"
+		(property "Reference" "R13"
 			(at 142.24 110.4899 0)
 			(show_name no)
@@
 			(project "EPICS_Connect4"
 				(path "/7f359823-7e50-4056-8b4f-ffb6c29ecc64/df1c4d5a-0179-43c9-baee-07d6baf032a1"
-					(reference "R14")
+					(reference "R13")
 					(unit 1)
 				)
@@
 		(dnp no)
 		(fields_autoplaced yes)
-		(property "Reference" "#PWR050"
+		(property "Reference" "#PWR048"
 			(at 228.6 118.11 0)
 			(hide yes)
@@
 			(project "EPICS_Connect4"
 				(path "/7f359823-7e50-4056-8b4f-ffb6c29ecc64/df1c4d5a-0179-43c9-baee-07d6baf032a1"
-					(reference "#PWR050")
+					(reference "#PWR048")
 					(unit 1)
 				)
@@
 		(dnp no)
 		(fields_autoplaced yes)
-		(property "Reference" "#PWR044"
+		(property "Reference" "#PWR042"
 			(at 152.4 113.03 0)
 			(hide yes)
@@
 			(project "EPICS_Connect4"
 				(path "/7f359823-7e50-4056-8b4f-ffb6c29ecc64/df1c4d5a-0179-43c9-baee-07d6baf032a1"
-					(reference "#PWR044")
+					(reference "#PWR042")
 					(unit 1)
 				)
@@
 		(dnp no)
 		(fields_autoplaced yes)
-		(property "Reference" "#PWR046"
+		(property "Reference" "#PWR044"
 			(at 177.8 80.01 0)
 			(hide yes)
@@
 			(project "EPICS_Connect4"
 				(path "/7f359823-7e50-4056-8b4f-ffb6c29ecc64/df1c4d5a-0179-43c9-baee-07d6baf032a1"
-					(reference "#PWR046")
+					(reference "#PWR044")
 					(unit 1)
 				)
@@
 		(body_style 1)
 		(exclude_from_sim no)
-		(in_bom yes)
+		(in_bom no)
 		(on_board yes)
 		(in_pos_files yes)
 		(dnp no)
-		(property "Reference" "TP13"
+		(property "Reference" "TP7"
 			(at 146.05 69.85 0)
 			(show_name no)
@@
 			(project "EPICS_Connect4"
 				(path "/7f359823-7e50-4056-8b4f-ffb6c29ecc64/df1c4d5a-0179-43c9-baee-07d6baf032a1"
-					(reference "TP13")
+					(reference "TP7")
 					(unit 1)
 				)
@@
 		(dnp no)
 		(fields_autoplaced yes)
-		(property "Reference" "R15"
+		(property "Reference" "R16"
 			(at 154.94 110.4899 0)
 			(show_name no)
@@
 			(project "EPICS_Connect4"
 				(path "/7f359823-7e50-4056-8b4f-ffb6c29ecc64/df1c4d5a-0179-43c9-baee-07d6baf032a1"
-					(reference "R15")
+					(reference "R16")
 					(unit 1)
 				)
@@
 		(dnp no)
 		(fields_autoplaced yes)
-		(property "Reference" "J3"
+		(property "Reference" "J8"
 			(at 60.96 81.28 0)
 			(show_name no)
@@
 			(project "EPICS_Connect4"
 				(path "/7f359823-7e50-4056-8b4f-ffb6c29ecc64/df1c4d5a-0179-43c9-baee-07d6baf032a1"
-					(reference "J3")
+					(reference "J8")
 					(unit 1)
 				)
@@
 		(dnp no)
 		(fields_autoplaced yes)
-		(property "Reference" "D3"
+		(property "Reference" "D5"
 			(at 231.14 120.5864 90)
 			(show_name no)
@@
 			(project "EPICS_Connect4"
 				(path "/7f359823-7e50-4056-8b4f-ffb6c29ecc64/df1c4d5a-0179-43c9-baee-07d6baf032a1"
-					(reference "D3")
+					(reference "D5")
 					(unit 1)
 				)
@@
 		(dnp no)
 		(fields_autoplaced yes)
-		(property "Reference" "#PWR042"
+		(property "Reference" "#PWR040"
 			(at 139.7 130.81 0)
 			(hide yes)
@@
 			(project "EPICS_Connect4"
 				(path "/7f359823-7e50-4056-8b4f-ffb6c29ecc64/df1c4d5a-0179-43c9-baee-07d6baf032a1"
-					(reference "#PWR042")
+					(reference "#PWR040")
 					(unit 1)
 				)
@@
 		(dnp no)
 		(fields_autoplaced yes)
-		(property "Reference" "#PWR037"
+		(property "Reference" "#PWR035"
 			(at 53.34 133.35 0)
 			(hide yes)
@@
 			(project "EPICS_Connect4"
 				(path "/7f359823-7e50-4056-8b4f-ffb6c29ecc64/df1c4d5a-0179-43c9-baee-07d6baf032a1"
-					(reference "#PWR037")
+					(reference "#PWR035")
 					(unit 1)
 				)
@@
 		(dnp no)
 		(fields_autoplaced yes)
-		(property "Reference" "#PWR045"
+		(property "Reference" "#PWR043"
 			(at 152.4 130.81 0)
 			(hide yes)
@@
 			(project "EPICS_Connect4"
 				(path "/7f359823-7e50-4056-8b4f-ffb6c29ecc64/df1c4d5a-0179-43c9-baee-07d6baf032a1"
-					(reference "#PWR045")
+					(reference "#PWR043")
 					(unit 1)
 				)
@@
 		(dnp no)
 		(fields_autoplaced yes)
-		(property "Reference" "#PWR043"
+		(property "Reference" "#PWR041"
 			(at 152.4 95.25 0)
 			(hide yes)
@@
 			(project "EPICS_Connect4"
 				(path "/7f359823-7e50-4056-8b4f-ffb6c29ecc64/df1c4d5a-0179-43c9-baee-07d6baf032a1"
-					(reference "#PWR043")
+					(reference "#PWR041")
 					(unit 1)
 				)
@@
 		(dnp no)
 		(fields_autoplaced yes)
-		(property "Reference" "R17"
+		(property "Reference" "R15"
 			(at 154.94 92.7099 0)
 			(show_name no)
@@
 			(project "EPICS_Connect4"
 				(path "/7f359823-7e50-4056-8b4f-ffb6c29ecc64/df1c4d5a-0179-43c9-baee-07d6baf032a1"
-					(reference "R17")
+					(reference "R15")
 					(unit 1)
 				)
@@
 		(body_style 1)
 		(exclude_from_sim no)
-		(in_bom yes)
+		(in_bom no)
 		(on_board yes)
 		(in_pos_files yes)
 		(dnp no)
-		(property "Reference" "TP14"
+		(property "Reference" "TP8"
 			(at 152.4 69.85 0)
 			(show_name no)
@@
 			(project "EPICS_Connect4"
 				(path "/7f359823-7e50-4056-8b4f-ffb6c29ecc64/df1c4d5a-0179-43c9-baee-07d6baf032a1"
-					(reference "TP14")
+					(reference "TP8")
 					(unit 1)
 				)
@@
 		(dnp no)
 		(fields_autoplaced yes)
-		(property "Reference" "#PWR049"
+		(property "Reference" "#PWR047"
 			(at 203.2 140.97 0)
 			(hide yes)
@@
 			(project "EPICS_Connect4"
 				(path "/7f359823-7e50-4056-8b4f-ffb6c29ecc64/df1c4d5a-0179-43c9-baee-07d6baf032a1"
-					(reference "#PWR049")
+					(reference "#PWR047")
 					(unit 1)
 				)
@@
 		(dnp no)
 		(fields_autoplaced yes)
-		(property "Reference" "#PWR041"
+		(property "Reference" "#PWR039"
 			(at 139.7 113.03 0)
 			(hide yes)
@@
 			(project "EPICS_Connect4"
 				(path "/7f359823-7e50-4056-8b4f-ffb6c29ecc64/df1c4d5a-0179-43c9-baee-07d6baf032a1"
-					(reference "#PWR041")
+					(reference "#PWR039")
 					(unit 1)
 				)
@@
 		(dnp no)
 		(fields_autoplaced yes)
-		(property "Reference" "C21"
+		(property "Reference" "C18"
 			(at 193.04 77.4699 0)
 			(show_name no)
@@
 			(project "EPICS_Connect4"
 				(path "/7f359823-7e50-4056-8b4f-ffb6c29ecc64/df1c4d5a-0179-43c9-baee-07d6baf032a1"
-					(reference "C21")
+					(reference "C18")
 					(unit 1)
 				)
@@
 		(dnp no)
 		(fields_autoplaced yes)
-		(property "Reference" "#PWR040"
+		(property "Reference" "#PWR038"
 			(at 139.7 95.25 0)
 			(hide yes)
@@
 			(project "EPICS_Connect4"
 				(path "/7f359823-7e50-4056-8b4f-ffb6c29ecc64/df1c4d5a-0179-43c9-baee-07d6baf032a1"
-					(reference "#PWR040")
+					(reference "#PWR038")
 					(unit 1)
 				)
@@
 		(in_pos_files yes)
 		(dnp no)
-		(property "Reference" "U7"
+		(property "Reference" "U4"
 			(at 90.5511 95.25 0)
 			(show_name no)
@@
 			(project "EPICS_Connect4"
 				(path "/7f359823-7e50-4056-8b4f-ffb6c29ecc64/df1c4d5a-0179-43c9-baee-07d6baf032a1"
-					(reference "U7")
+					(reference "U4")
 					(unit 1)
 				)
@@
 		(dnp no)
 		(fields_autoplaced yes)
-		(property "Reference" "R13"
+		(property "Reference" "R17"
 			(at 231.14 115.5699 0)
 			(show_name no)
@@
 			(project "EPICS_Connect4"
 				(path "/7f359823-7e50-4056-8b4f-ffb6c29ecc64/df1c4d5a-0179-43c9-baee-07d6baf032a1"
-					(reference "R13")
+					(reference "R17")
 					(unit 1)
 				)
@@
 		(dnp no)
 		(fields_autoplaced yes)
-		(property "Reference" "#PWR048"
+		(property "Reference" "#PWR046"
 			(at 177.8 105.41 0)
 			(hide yes)
@@
 			(project "EPICS_Connect4"
 				(path "/7f359823-7e50-4056-8b4f-ffb6c29ecc64/df1c4d5a-0179-43c9-baee-07d6baf032a1"
-					(reference "#PWR048")
+					(reference "#PWR046")
 					(unit 1)
 				)
