File: PCB/esp32.kicad_sch (KiCad schematic)
At the start: 21 parts, among them J8 USB_C_Receptacle_USB2.0_14P, SW1 ESP.RST, SW2 ESP.BOOT, U4 USBLC6-2SC6, U7 ESP32-C3-WROOM-02

Commit message: Ready for Fab
Parts:
- renumbered U7 to U5, U4 to U6
Changed lines of the file:
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@@
 		(dnp no)
 		(fields_autoplaced yes)
-		(property "Reference" "U7"
+		(property "Reference" "U5"
 			(at 205.3433 86.36 0)
 			(show_name no)
@@
 			(project "EPICS_Connect4"
 				(path "/7f359823-7e50-4056-8b4f-ffb6c29ecc64/df1c4d5a-0179-43c9-baee-07d6baf032a1"
-					(reference "U7")
+					(reference "U5")
 					(unit 1)
 				)
@@
 		(in_pos_files yes)
 		(dnp no)
-		(property "Reference" "U4"
+		(property "Reference" "U6"
 			(at 90.5511 95.25 0)
 			(show_name no)
@@
 			(project "EPICS_Connect4"
 				(path "/7f359823-7e50-4056-8b4f-ffb6c29ecc64/df1c4d5a-0179-43c9-baee-07d6baf032a1"
-					(reference "U4")
+					(reference "U6")
 					(unit 1)
 				)
