File: PCB/motor.kicad_sch (KiCad schematic)
At the start: 3 parts, among them U7 TMC2209

Commit message: Update EPICS_Connect4 KiCad project
Co-Authored-By: Claude Sonnet 5 <noreply@anthropic.com>
Parts:
- U8: renamed from U7; footprint (none) -> Library:STEPSTICK_socket
Changed lines of the file:
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@@
 		)
 	)
-	(hierarchical_label "M1"
+	(hierarchical_label "M1[3..0]"
 		(shape output)
 		(at 177.8 76.2 90)
@@
 		(in_pos_files yes)
 		(dnp no)
-		(property "Reference" "#PWR?"
+		(property "Reference" "#PWR067"
 			(at 165.1 87.63 0)
 			(hide yes)
@@
 			(project "EPICS_Connect4"
 				(path "/7f359823-7e50-4056-8b4f-ffb6c29ecc64/8848091b-3b50-4b93-b829-b49cad79e851"
-					(reference "#PWR?")
+					(reference "#PWR067")
 					(unit 1)
 				)
@@
 		(in_pos_files yes)
 		(dnp no)
-		(property "Reference" "#PWR?"
+		(property "Reference" "#PWR066"
 			(at 154.94 143.51 0)
 			(hide yes)
@@
 			(project "EPICS_Connect4"
 				(path "/7f359823-7e50-4056-8b4f-ffb6c29ecc64/8848091b-3b50-4b93-b829-b49cad79e851"
-					(reference "#PWR?")
+					(reference "#PWR066")
 					(unit 1)
 				)
@@
 		(in_pos_files yes)
 		(dnp no)
-		(property "Reference" "#PWR?"
+		(property "Reference" "#PWR061"
 			(at 139.7 87.63 0)
 			(hide yes)
@@
 			(project "EPICS_Connect4"
 				(path "/7f359823-7e50-4056-8b4f-ffb6c29ecc64/8848091b-3b50-4b93-b829-b49cad79e851"
-					(reference "#PWR?")
+					(reference "#PWR061")
 					(unit 1)
 				)
@@
 		(dnp no)
 		(fields_autoplaced yes)
-		(property "Reference" "#PWR?"
+		(property "Reference" "#PWR062"
 			(at 133.35 109.22 0)
 			(hide yes)
@@
 			(project "EPICS_Connect4"
 				(path "/7f359823-7e50-4056-8b4f-ffb6c29ecc64/8848091b-3b50-4b93-b829-b49cad79e851"
-					(reference "#PWR?")
+					(reference "#PWR062")
 					(unit 1)
 				)
@@
 		(in_pos_files yes)
 		(dnp no)
-		(property "Reference" "U7"
+		(property "Reference" "U8"
 			(at 151.13 85.09 0)
 			(show_name no)
@@
 			)
 		)
-		(property "Footprint" ""
+		(property "Footprint" "Library:STEPSTICK_socket"
 			(at 139.7 85.09 0)
 			(hide yes)
@@
 			(project "EPICS_Connect4"
 				(path "/7f359823-7e50-4056-8b4f-ffb6c29ecc64/8848091b-3b50-4b93-b829-b49cad79e851"
-					(reference "U7")
+					(reference "U8")
 					(unit 1)
 				)
@@
 		(in_pos_files yes)
 		(dnp no)
-		(property "Reference" "#PWR?"
+		(property "Reference" "#PWR065"
 			(at 152.4 127 0)
 			(hide yes)
@@
 			(project "EPICS_Connect4"
 				(path "/7f359823-7e50-4056-8b4f-ffb6c29ecc64/8848091b-3b50-4b93-b829-b49cad79e851"
-					(reference "#PWR?")
+					(reference "#PWR065")
 					(unit 1)
 				)
@@
 		(dnp no)
 		(fields_autoplaced yes)
-		(property "Reference" "#PWR?"
+		(property "Reference" "#PWR063"
 			(at 148.59 82.55 0)
 			(hide yes)
@@
 			(project "EPICS_Connect4"
 				(path "/7f359823-7e50-4056-8b4f-ffb6c29ecc64/8848091b-3b50-4b93-b829-b49cad79e851"
-					(reference "#PWR?")
+					(reference "#PWR063")
 					(unit 1)
 				)
@@
 		(in_pos_files yes)
 		(dnp no)
-		(property "Reference" "#PWR?"
+		(property "Reference" "#PWR064"
 			(at 149.86 143.51 0)
 			(hide yes)
@@
 			(project "EPICS_Connect4"
 				(path "/7f359823-7e50-4056-8b4f-ffb6c29ecc64/8848091b-3b50-4b93-b829-b49cad79e851"
-					(reference "#PWR?")
-					(unit 1)
-				)
+					(reference "#PWR064")
+					(unit 1)
+				)

Commit message: Swap Molex connector 3D model to 43650-0215
Co-Authored-By: Claude Opus 5.5 <noreply@anthropic.com>
Parts:
- renumbered C22 to C20, C23 to C21, U8 to U5
Changed lines of the file:
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@@
 		(in_pos_files yes)
 		(dnp no)
-		(property "Reference" "#PWR067"
+		(property "Reference" "#PWR059"
 			(at 165.1 87.63 0)
 			(hide yes)
@@
 			(project "EPICS_Connect4"
 				(path "/7f359823-7e50-4056-8b4f-ffb6c29ecc64/8848091b-3b50-4b93-b829-b49cad79e851"
-					(reference "#PWR067")
+					(reference "#PWR059")
 					(unit 1)
 				)
@@
 		(in_pos_files yes)
 		(dnp no)
-		(property "Reference" "C23"
+		(property "Reference" "C21"
 			(at 161.29 74.93 90)
 			(show_name no)
@@
 			(project "EPICS_Connect4"
 				(path "/7f359823-7e50-4056-8b4f-ffb6c29ecc64/8848091b-3b50-4b93-b829-b49cad79e851"
-					(reference "C23")
+					(reference "C21")
 					(unit 1)
 				)
@@
 		(in_pos_files yes)
 		(dnp no)
-		(property "Reference" "#PWR066"
+		(property "Reference" "#PWR058"
 			(at 154.94 143.51 0)
 			(hide yes)
@@
 			(project "EPICS_Connect4"
 				(path "/7f359823-7e50-4056-8b4f-ffb6c29ecc64/8848091b-3b50-4b93-b829-b49cad79e851"
-					(reference "#PWR066")
+					(reference "#PWR058")
 					(unit 1)
 				)
@@
 		(in_pos_files yes)
 		(dnp no)
-		(property "Reference" "#PWR061"
+		(property "Reference" "#PWR053"
 			(at 139.7 87.63 0)
 			(hide yes)
@@
 			(project "EPICS_Connect4"
 				(path "/7f359823-7e50-4056-8b4f-ffb6c29ecc64/8848091b-3b50-4b93-b829-b49cad79e851"
-					(reference "#PWR061")
+					(reference "#PWR053")
 					(unit 1)
 				)
@@
 		(dnp no)
 		(fields_autoplaced yes)
-		(property "Reference" "C22"
+		(property "Reference" "C20"
 			(at 143.51 74.93 90)
 			(show_name no)
@@
 			(project "EPICS_Connect4"
 				(path "/7f359823-7e50-4056-8b4f-ffb6c29ecc64/8848091b-3b50-4b93-b829-b49cad79e851"
-					(reference "C22")
+					(reference "C20")
 					(unit 1)
 				)
@@
 		(dnp no)
 		(fields_autoplaced yes)
-		(property "Reference" "#PWR062"
+		(property "Reference" "#PWR054"
 			(at 133.35 109.22 0)
 			(hide yes)
@@
 			(project "EPICS_Connect4"
 				(path "/7f359823-7e50-4056-8b4f-ffb6c29ecc64/8848091b-3b50-4b93-b829-b49cad79e851"
-					(reference "#PWR062")
+					(reference "#PWR054")
 					(unit 1)
 				)
@@
 		(in_pos_files yes)
 		(dnp no)
-		(property "Reference" "U8"
+		(property "Reference" "U5"
 			(at 151.13 85.09 0)
 			(show_name no)
@@
 			(project "EPICS_Connect4"
 				(path "/7f359823-7e50-4056-8b4f-ffb6c29ecc64/8848091b-3b50-4b93-b829-b49cad79e851"
-					(reference "U8")
+					(reference "U5")
 					(unit 1)
 				)
@@
 		(in_pos_files yes)
 		(dnp no)
-		(property "Reference" "#PWR065"
+		(property "Reference" "#PWR057"
 			(at 152.4 127 0)
 			(hide yes)
@@
 			(project "EPICS_Connect4"
 				(path "/7f359823-7e50-4056-8b4f-ffb6c29ecc64/8848091b-3b50-4b93-b829-b49cad79e851"
-					(reference "#PWR065")
+					(reference "#PWR057")
 					(unit 1)
 				)
@@
 		(dnp no)
 		(fields_autoplaced yes)
-		(property "Reference" "#PWR063"
+		(property "Reference" "#PWR055"
 			(at 148.59 82.55 0)
 			(hide yes)
@@
 			(project "EPICS_Connect4"
 				(path "/7f359823-7e50-4056-8b4f-ffb6c29ecc64/8848091b-3b50-4b93-b829-b49cad79e851"
-					(reference "#PWR063")
+					(reference "#PWR055")
 					(unit 1)
 				)
@@
 		(in_pos_files yes)
 		(dnp no)
-		(property "Reference" "#PWR064"
+		(property "Reference" "#PWR056"
 			(at 149.86 143.51 0)
 			(hide yes)
@@
 			(project "EPICS_Connect4"
 				(path "/7f359823-7e50-4056-8b4f-ffb6c29ecc64/8848091b-3b50-4b93-b829-b49cad79e851"
-					(reference "#PWR064")
-					(unit 1)
-				)
+					(reference "#PWR056")
+					(unit 1)
+				)
