File: PCB/motor.kicad_sch (KiCad schematic)
At the start: 3 parts, among them U5 TMC2209

Commit message: Ready for Fab
Parts:
- renumbered U5 to U7
Changed lines of the file:
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@@
 		(in_pos_files yes)
 		(dnp no)
-		(property "Reference" "U5"
+		(property "Reference" "U7"
 			(at 151.13 85.09 0)
 			(show_name no)
@@
 			(project "EPICS_Connect4"
 				(path "/7f359823-7e50-4056-8b4f-ffb6c29ecc64/8848091b-3b50-4b93-b829-b49cad79e851"
-					(reference "U5")
+					(reference "U7")
 					(unit 1)
 				)
