File: PCB/power.kicad_sch (KiCad schematic)
At the start: 13 parts, among them U1 TPS54202DDC, U2 AP2205-5

Commit message: Minor PCB updates
Co-Authored-By: Claude Sonnet 5 <noreply@anthropic.com>
Parts:
- U1: footprint Package_TO_SOT_SMD:SOT-23-6 -> Package_TO_SOT_SMD:SOT-23-6_Handsoldering
- U2: footprint Package_TO_SOT_SMD:SOT-23-5 -> Package_TO_SOT_SMD:SOT-23-5_HandSoldering
Changed lines of the file:
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@@
 			)
 		)
-		(property "Footprint" "Package_TO_SOT_SMD:SOT-23-5"
+		(property "Footprint" "Package_TO_SOT_SMD:SOT-23-5_HandSoldering"
 			(at 152.4 121.285 0)
 			(hide yes)
@@
 			)
 		)
-		(property "Footprint" "Package_TO_SOT_SMD:SOT-23-6"
+		(property "Footprint" "Package_TO_SOT_SMD:SOT-23-6_Handsoldering"
 			(at 153.67 100.33 0)
 			(hide yes)

Commit message: Swap Molex connector 3D model to 43650-0215
Co-Authored-By: Claude Opus 5.5 <noreply@anthropic.com>
Parts:
- removed C7: 1uF, Capacitor_SMD:C_0603_1608Metric, symbol Device:C_Small
- removed C8: 10uF, Capacitor_SMD:C_0603_1608Metric, symbol Device:C_Small
- removed U2: AP2205-5, Package_TO_SOT_SMD:SOT-23-5_HandSoldering, symbol Connect4_Library:AP2205-5
- C2: value 10uF -> 22uF
Connections:
- net +12V renamed +VIN
Other:
- note removed: "SECONDARY +5V LOGIC SHIFTER SUPPLY"
