File: PCB/stm32.kicad_sch (KiCad schematic)
At the start: 27 parts, among them J2 TC2030, U3 SN74AHCT1G125DBVR, U4 SN74AHCT1G125DBVR

Commit message: Update EPICS_Connect4 KiCad project
Co-Authored-By: Claude Sonnet 5 <noreply@anthropic.com>
Parts:
- gave numbers to parts that had none: 1
- renumbered U3 to U4, U4 to U5
Connections:
- net +3V3: now also D2.2 (A); no longer R10.1
- net U_LED: now also R10.2, U3.17 (PB1); no longer D2.1 (K), U3.33 (PA11)
- new net: D2.1 (K), R10.1
Other:
- moved on the sheet: D2, R10

Commit message: Update PCB layout
Co-Authored-By: Claude Sonnet 5 <noreply@anthropic.com>
Connections:
- net ledDataA: now also TP8.1
- net ledDataB: now also TP9.1
- net at R12.1, U5.4 (Y): no longer TP9.1
- net at R11.1, U4.4 (Y): no longer TP8.1
Other:
- moved on the sheet: TP8, TP9

Commit message: Swap Molex connector 3D model to 43650-0215
Co-Authored-By: Claude Opus 5.5 <noreply@anthropic.com>
Parts:
- added TP2, TP4: GND, TestPoint:TestPoint_Pad_1.0x1.0mm, symbol Connector:TestPoint
- TP1: renamed from TP7; now left out of the parts list
- TP3: renamed from TP8; now left out of the parts list
- TP5: renamed from TP9; now left out of the parts list
- renumbered C12 to C10, C13 to C11, C14 to C12, C15 to C13, C16 to C14, C17 to C15, C18 to C16, C9 to C7, C10 to C8, C11 to C9, D2 to D4, J2 to J9, R7 to R10, R8 to R4, R9 to R5, R10 to R6, R4 to R7, R5 to R8, R6 to R9, U4 to U2, U5 to U3, U3 to U6
Connections:
- net GND: now also TP2.1, TP4.1
