File: PCB/stm32.kicad_sch (KiCad schematic)
At the start: 29 parts, among them J9 TC2030, U2 SN74AHCT1G125DBVR, U3 SN74AHCT1G125DBVR, U6 STM32G474CBTx

Commit message: Ready for Fab
Parts:
- renumbered U6 to U2, U2 to U3, U3 to U4
Changed lines of the file:
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@@
 		(in_pos_files yes)
 		(dnp no)
-		(property "Reference" "U3"
+		(property "Reference" "U4"
 			(at 215.9 110.49 0)
 			(show_name no)
@@
 			(project "EPICS_Connect4"
 				(path "/7f359823-7e50-4056-8b4f-ffb6c29ecc64/44155fe5-a28f-41a7-abb9-b121067c4744"
-					(reference "U3")
+					(reference "U4")
 					(unit 1)
 				)
@@
 		(in_pos_files yes)
 		(dnp no)
-		(property "Reference" "U2"
+		(property "Reference" "U3"
 			(at 215.9 72.39 0)
 			(show_name no)
@@
 			(project "EPICS_Connect4"
 				(path "/7f359823-7e50-4056-8b4f-ffb6c29ecc64/44155fe5-a28f-41a7-abb9-b121067c4744"
-					(reference "U2")
+					(reference "U3")
 					(unit 1)
 				)
@@
 		(dnp no)
 		(fields_autoplaced yes)
-		(property "Reference" "U6"
+		(property "Reference" "U2"
 			(at 157.0833 144.78 0)
 			(show_name no)
@@
 			(project "EPICS_Connect4"
 				(path "/7f359823-7e50-4056-8b4f-ffb6c29ecc64/44155fe5-a28f-41a7-abb9-b121067c4744"
-					(reference "U6")
+					(reference "U2")
 					(unit 1)
 				)
